Commit message: xacro clean-up in progress

File: urdf/m2xr.xacro (robot description, xacro)
@@ -1,53 +1,6 @@
 <?xml version="1.0"?>
 <robot name="m2wr" xmlns:xacro="http://ros.org/wiki/xacro">
-  <material name="black">
-    <color rgba="0.0 0.0 0.0 1.0"/>
-  </material>
-  <material name="blue">
-    <color rgba="0.203125 0.23828125 0.28515625 1.0"/>
-  </material>
-  <material name="green">
-    <color rgba="0.0 0.8 0.0 1.0"/>
-  </material>
-  <material name="grey">
-    <color rgba="0.2 0.2 0.2 1.0"/>
-  </material>
-  <material name="orange">
-    <color rgba="1.0 0.423529411765 0.0392156862745 1.0"/>
-  </material>
-  <material name="brown">
-    <color rgba="0.870588235294 0.811764705882 0.764705882353 1.0"/>
-  </material>
-  <material name="red">
-    <color rgba="0.80078125 0.12890625 0.1328125 1.0"/>
-  </material>
-  <material name="white">
-    <color rgba="1.0 1.0 1.0 1.0"/>
-  </material>
-  <gazebo reference="link_chassis">
-    <material>Gazebo/Orange</material>
-  </gazebo>
-  <gazebo reference="link_left_wheel">
-    <material>Gazebo/Blue</material>
-  </gazebo>
-  <gazebo reference="link_right_wheel">
-    <material>Gazebo/Blue</material>
-  </gazebo>
-  <gazebo>
-    <plugin filename="libgazebo_ros_diff_drive.so" name="differential_drive_controller">
-      <legacyMode>false</legacyMode>
-      <alwaysOn>true</alwaysOn>
-      <updateRate>20</updateRate>
-      <leftJoint>joint_left_wheel</leftJoint>
-      <rightJoint>joint_right_wheel</rightJoint>
-      <wheelSeparation>0.2</wheelSeparation>
-      <wheelDiameter>0.2</wheelDiameter>
-      <torque>0.1</torque>
-      <commandTopic>cmd_vel</commandTopic>
-      <odometryTopic>odom</odometryTopic>
-      <odometryFrame>odom</odometryFrame>
-      <robotBaseFrame>link_chassis</robotBaseFrame>
-    </plugin>
-  </gazebo>
+	<xacro:include filename="$(find ros_diff_drive)/urdf/materials.xacro" />
+	<xacro:include filename="$(find ros_diff_drive)/urdf/gazebo_macros.gazebo" />
   <link name="link_chassis">
     <!-- pose and inertial -->

Commit message: Created macro for wheel links

File: urdf/m2xr.xacro (robot description, xacro)
@@ -3,4 +3,5 @@
 	<xacro:include filename="$(find ros_diff_drive)/urdf/materials.xacro" />
 	<xacro:include filename="$(find ros_diff_drive)/urdf/gazebo_macros.gazebo" />
+  <xacro:include filename="$(find ros_diff_drive)/urdf/macros.xacro"/>
   <link name="link_chassis">
     <!-- pose and inertial -->
@@ -48,23 +49,6 @@
     </visual>
   </link>
-  <link name="link_right_wheel">
-    <inertial>
-      <mass value="0.2"/>
-      <origin rpy="0 1.5707 1.5707" xyz="0 0 0"/>
-      <inertia ixx="0.000526666666667" ixy="0" ixz="0" iyy="0.000526666666667" iyz="0" izz="0.001"/>
-    </inertial>
-    <collision name="link_right_wheel_collision">
-      <origin rpy="0 1.5707 1.5707" xyz="0 0 0"/>
-      <geometry>
-        <cylinder length="0.04" radius="0.1"/>
-      </geometry>
-    </collision>
-    <visual name="link_right_wheel_visual">
-      <origin rpy="0 1.5707 1.5707" xyz="0 0 0"/>
-      <geometry>
-        <cylinder length="0.04" radius="0.1"/>
-      </geometry>
-    </visual>
-  </link>
+<xacro:link_wheel wheel_name="link_right_wheel" />
+<xacro:link_wheel wheel_name="link_left_wheel" />
   <joint name="joint_right_wheel" type="continuous">
     <origin rpy="0 0 0" xyz="-0.05 0.15 0"/>
@@ -75,23 +59,4 @@
     <joint_properties damping="1.0" friction="1.0"/>
   </joint>
-  <link name="link_left_wheel">
-    <inertial>
-      <mass value="0.2"/>
-      <origin rpy="0 1.5707 1.5707" xyz="0 0 0"/>
-      <inertia ixx="0.000526666666667" ixy="0" ixz="0" iyy="0.000526666666667" iyz="0" izz="0.001"/>
-    </inertial>
-    <collision name="link_left_wheel_collision">
-      <origin rpy="0 1.5707 1.5707" xyz="0 0 0"/>
-      <geometry>
-        <cylinder length="0.04" radius="0.1"/>
-      </geometry>
-    </collision>
-    <visual name="link_left_wheel_visual">
-      <origin rpy="0 1.5707 1.5707" xyz="0 0 0"/>
-      <geometry>
-        <cylinder length="0.04" radius="0.1"/>
-      </geometry>
-    </visual>
-  </link>
   <joint name="joint_left_wheel" type="continuous">
     <origin rpy="0 0 0" xyz="-0.05 -0.15 0"/>

Commit message: New macros introduced

File: urdf/m2xr.xacro (robot description, xacro)
@@ -15,5 +15,5 @@
     <collision name="collision_chassis">
       <geometry>
-        <box size="0.5 0.3 0.07"/>
+        <xacro:chasis_geometry_box/>
       </geometry>
     </collision>
@@ -21,5 +21,5 @@
       <origin rpy="0 0 0" xyz="0 0 0"/>
       <geometry>
-        <box size="0.5 0.3 0.07"/>
+        <xacro:chasis_geometry_box/>
       </geometry>
       <material name="blue"/>
@@ -52,5 +52,5 @@
 <xacro:link_wheel wheel_name="link_left_wheel" />
   <joint name="joint_right_wheel" type="continuous">
-    <origin rpy="0 0 0" xyz="-0.05 0.15 0"/>
+    <origin rpy="0 0 0" xyz="-0.05 ${chassis_box_wid/2.0} 0"/>
     <child link="link_right_wheel"/>
     <parent link="link_chassis"/>
@@ -60,5 +60,5 @@
   </joint>
   <joint name="joint_left_wheel" type="continuous">
-    <origin rpy="0 0 0" xyz="-0.05 -0.15 0"/>
+    <origin rpy="0 0 0" xyz="-0.05 -${chassis_box_wid/2.0} 0"/>
     <child link="link_left_wheel"/>
     <parent link="link_chassis"/>

File: urdf/macros.xacro (robot description, xacro)
@@ -1,4 +1,9 @@
 <?xml version="1.0"?>
 <robot xmlns:xacro="http://wiki.ros.org/xacro">
+  <xacro:property name="chassis_box_len" value="0.5"/>
+  <xacro:property name="chassis_box_wid" value="0.3"/>
+  <xacro:property name="chassis_box_hgt" value="0.07"/>
+  <xacro:property name="odom_wheel_radius" value="0.1"/>
+  <xacro:property name="odom_wheel_len" value="0.04"/>
   <xacro:macro name="link_wheel" params="wheel_name">
     <link name="${wheel_name}">
@@ -11,5 +16,5 @@
         <origin rpy="0 1.5707 1.5707" xyz="0 0 0"/>
         <geometry>
-          <cylinder length="0.04" radius="0.1"/>
+          <cylinder length="${odom_wheel_len}" radius="${odom_wheel_radius}"/>
         </geometry>
       </collision>
@@ -17,8 +22,11 @@
       <origin rpy="0 1.5707 1.5707" xyz="0 0 0"/>
         <geometry>
-          <cylinder length="0.04" radius="0.1"/>
+          <cylinder length="${odom_wheel_len}" radius="${odom_wheel_radius}"/>
         </geometry>
       </visual>
     </link>
   </xacro:macro>
+  <xacro:macro name="chasis_geometry_box">
+    <box size="${chassis_box_len} ${chassis_box_wid} ${chassis_box_hgt}"/>
+  </xacro:macro>
 </robot>

Commit message: wheel joints parametarised

File: urdf/m2xr.xacro (robot description, xacro)
@@ -49,23 +49,9 @@
     </visual>
   </link>
-<!-- Right and left wheels -->
-<xacro:link_wheel wheel_name="link_right_wheel" />
-<xacro:link_wheel wheel_name="link_left_wheel" />
+  <!-- Right and left wheels -->
+  <xacro:link_wheel wheel_name="link_right_wheel" />
+  <xacro:link_wheel wheel_name="link_left_wheel" />
   <!-- Right and left joints -->
-  <joint name="joint_right_wheel" type="continuous">
-    <origin rpy="0 0 0" xyz="-0.05 ${chassis_box_wid/2.0} 0"/>
-    <child link="link_right_wheel"/>
-    <parent link="link_chassis"/>
-    <axis rpy="0 0 0" xyz="0 1 0"/>
-    <limit effort="10000" velocity="1000"/>
-    <joint_properties damping="1.0" friction="1.0"/>
-  </joint>
-  <joint name="joint_left_wheel" type="continuous">
-    <origin rpy="0 0 0" xyz="-0.05 -${chassis_box_wid/2.0} 0"/>
-    <child link="link_left_wheel"/>
-    <parent link="link_chassis"/>
-    <axis rpy="0 0 0" xyz="0 1 0"/>
-    <limit effort="10000" velocity="1000"/>
-    <joint_properties damping="1.0" friction="1.0"/>
-  </joint>
+  <xacro:joint_wheel name="joint_right_wheel" child="link_right_wheel" origin_xyz="-0.05 ${chassis_box_wid/2.0} 0"/>
+  <xacro:joint_wheel name="joint_left_wheel" child="link_left_wheel" origin_xyz="-0.05 -${chassis_box_wid/2.0} 0"/>
 </robot>

File: urdf/macros.xacro (robot description, xacro)
@@ -27,4 +27,14 @@
     </link>
   </xacro:macro>
+  <xacro:macro name="joint_wheel" params="name child origin_xyz">
+    <joint name="${name}" type="continuous">
+      <origin rpy="0 0 0" xyz="${origin_xyz}"/>
+      <child link="${child}"/>
+      <parent link="link_chassis"/>
+      <axis rpy="0 0 0" xyz="0 1 0"/>
+      <limit effort="10000" velocity="1000"/>
+      <joint_properties damping="1.0" friction="1.0"/>
+    </joint>
+  </xacro:macro>
   <xacro:macro name="chasis_geometry_box">
     <box size="${chassis_box_len} ${chassis_box_wid} ${chassis_box_hgt}"/>
